Commit message: Feat: Fix kistar_hand urdf & Add usd file for isaacsim 5.x.x

File: robots/hands/kistar_hand/kistar_hand.urdf (robot description, URDF)
Before this commit: robot kistar_hand, 34 links, 33 joints
Links:
- link kistar_hand_index_sensor_0: geometry visual mesh filename=meshes/kistar_hand_index_sensor_0_visuals.obj scale=1. 1. 1.
- link kistar_hand_index_sensor_1: geometry visual mesh filename=meshes/kistar_hand_index_sensor_1_visuals.obj scale=1. 1. 1.
- link kistar_hand_index_sensor_2: geometry visual mesh filename=meshes/kistar_hand_index_sensor_2_visuals.obj scale=1. 1. 1.
- link kistar_hand_middle_sensor_0: geometry visual mesh filename=meshes/kistar_hand_middle_sensor_0_visuals.obj scale=1. 1. 1.
- link kistar_hand_middle_sensor_1: geometry visual mesh filename=meshes/kistar_hand_middle_sensor_1_visuals.obj scale=1. 1. 1.
- link kistar_hand_middle_sensor_2: geometry visual mesh filename=meshes/kistar_hand_middle_sensor_2_visuals.obj scale=1. 1. 1.
- link kistar_hand_ring_sensor_0: geometry visual mesh filename=meshes/kistar_hand_ring_sensor_0_visuals.obj scale=1. 1. 1.
- link kistar_hand_ring_sensor_1: geometry visual mesh filename=meshes/kistar_hand_ring_sensor_1_visuals.obj scale=1. 1. 1.
- link kistar_hand_ring_sensor_2: geometry visual mesh filename=meshes/kistar_hand_ring_sensor_2_visuals.obj scale=1. 1. 1.
- link kistar_hand_thumb_sensor_0: geometry visual mesh filename=meshes/kistar_hand_thumb_sensor_0_visuals.obj scale=1. 1. 1.
- link kistar_hand_thumb_sensor_1: geometry visual mesh filename=meshes/kistar_hand_thumb_sensor_1_visuals.obj scale=1. 1. 1.
- link middle_basemotor: geometry visual mesh filename=meshes/middle_basemotor_visuals.obj scale=1. 1. 1.
- link middle_link_0: geometry visual mesh filename=meshes/middle_link_0_visuals.obj scale=1. 1. 1.
- link ring_basemotor: geometry visual mesh filename=meshes/ring_basemotor_visuals.obj scale=1. 1. 1.
- link ring_link_0: geometry visual mesh filename=meshes/ring_link_0_visuals.obj scale=1. 1. 1.
- link thumb_basemotor: geometry visual mesh filename=meshes/thumb_basemotor_visuals.obj scale=1. 1. 1.
- link thumb_link_0: geometry visual mesh filename=meshes/thumb_link_0_visuals.obj scale=1. 1. 1.
